Commit message: Added topic names as parameters in the launchfile, fixed namespacing.

File: z1_pro_driver/urdf/z1_pro_camera.urdf (robot description, URDF)
Before this commit: robot z1_pro_camera, 5 links, 4 joints
Links:
- removed link /gimbal_base
- removed link /gimbal_pitch_link
- removed link /gimbal_roll_link
- removed link /gimbal_yaw_link
- added link /base, mass 0.5; visual cylinder length=0.02 radius=0.03
- added link /pitch_link; visual box size=0.02 0.02 0.02
- added link /roll_link; visual box size=0.03 0.03 0.03
- added link /yaw_link; visual box size=0.02 0.02 0.02
Joints:
- removed joint gimbal_pitch_joint
- removed joint gimbal_roll_joint
- removed joint gimbal_yaw_joint
- added joint pitch_joint: type revolute, parent /roll_link, child /pitch_link, origin xyz=0.02096 0.0194 0.00736 rpy=0 0.3490 0, axis 0 1 0, limit lower=-1.5708 upper=1.5708 effort=1.0 velocity=2.0
- added joint roll_joint: type revolute, parent /yaw_link, child /roll_link, origin xyz=-0.01127 0 0.02163 rpy=0 -0.3490 0, axis 1 0 0, limit lower=-1.5708 upper=1.5708 effort=1.0 velocity=2.0
- added joint yaw_joint: type revolute, parent /base, child /yaw_link, origin xyz=0 0 0 rpy=0 0 0, axis 0 0 1, limit lower=-3.14159 upper=3.14159 effort=1.0 velocity=2.0
- joint camera_joint: parent /gimbal_pitch_link -> /pitch_link

Commit message: Add optical frame and joint to camera URDF

File: z1_pro_driver/urdf/z1_pro_camera.urdf (robot description, URDF)
Before this commit: robot z1_pro_camera, 5 links, 4 joints
Links:
- added link z1_optical_frame
Joints:
- added joint optical_joint: type fixed, parent z1_camera_link, child z1_optical_frame, origin xyz=0 0 0 rpy=-1.57079632679 0 -1.57079632679
